Commit message: changed robot base, fixed namespace for camera and imu, started porting localization

File: summit_xl_description/robots/summit_xls_icclab.urdf.xacro (robot description, xacro)
@@ -6,5 +6,5 @@
 	<!-- First we import all posible elements defined in the urdf.xacro files. All these elements are defined as macro:xacros -->
 	<!-- Import summit XL base elements -->
-	<xacro:include filename="$(find summit_xl_description)/urdf/bases/summit_xls_base.urdf.xacro" />
+	<xacro:include filename="$(find summit_xl_description)/urdf/bases/summit_xl_hls_base.urdf.xacro" />
 	<!-- Import summit XL wheels -->
 	<xacro:include filename="$(find summit_xl_description)/urdf/wheels/omni_wheel.urdf.xacro" />
@@ -52,5 +52,5 @@
 		<!-- Here we create the robot elements using the xacro:macros imported at the beggining of this file -->
 		<!-- Summit XL base -->
-		<xacro:summit_xls_base prefix="$(arg prefix)" publish_bf="true" hq="${hq}" />
+		<xacro:summit_xl_hls_base prefix="$(arg prefix)" publish_bf="true" hq="${hq}" />
 		<xacro:omni_wheel prefix="$(arg prefix)front_right" parent="$(arg prefix)base_link" reflect="false" hq="${hq}">
 			<origin xyz="${wheel_offset_x} -${wheel_offset_y} ${wheel_offset_z}" rpy="0 0 0"/>
@@ -66,7 +66,7 @@
 		</xacro:omni_wheel>
         <!-- IMU -->
-		<xacro:sensor_imu prefix="$(arg prefix)imu" parent="$(arg prefix)base_link">
+		<xacro:sensor_imu_hector prefix="$(arg prefix)imu" ns="$(arg robot_ns)" parent="$(arg prefix)base_link">
 			<origin xyz="${imu_offset_x} ${imu_offset_y} ${imu_offset_z}" rpy="0 0 0"/>
-		</xacro:sensor_imu>
+		</xacro:sensor_imu_hector>
 		<!-- SENSORS -->
 		<xacro:sensor_hokuyo_ust20lx ns="$(arg robot_ns)" prefix="front_laser" parent="base_link">
@@ -82,5 +82,5 @@
 			<origin xyz="${rear_ptz_camera_offset_x} ${rear_ptz_camera_offset_y} ${rear_ptz_camera_offset_z}" rpy="${-PI/2} 0 ${PI}"/>
 		</xacro:sensor_axis_m5013-->
-		<xacro:sensor_orbbec_astra prefix="$(arg prefix)front_rgbd_camera" parent="$(arg prefix)base_link" ns="front_rgbd_camera">
+		<xacro:sensor_orbbec_astra prefix="$(arg prefix)front_rgbd_camera" parent="$(arg prefix)base_link" ns="$(arg robot_ns)">
 			<origin xyz="${front_rgbd_camera_offset_x} ${front_rgbd_camera_offset_y} ${front_rgbd_camera_offset_z}" rpy="0 0 0"/>
 		</xacro:sensor_orbbec_astra>

File: summit_xl_description/urdf/bases/summit_xl_base.gazebo.xacro (robot description, xacro)
@@ -54,5 +54,5 @@
         <publish_rate>100</publish_rate>
         <publish_odom>true</publish_odom>
-        <publish_odom_tf>true</publish_odom_tf>
+        <publish_odom_tf>${publish_tf}</publish_odom_tf>
         <odometry_frame>${namespace}/odom</odometry_frame>
         <robot_base_frame>${namespace}/base_footprint</robot_base_frame>

File: summit_xl_description/urdf/bases/summit_xl_hls_base.urdf.xacro (robot description, xacro)
@@ -6,4 +6,5 @@
 	  <xacro:property name="PI" value="3.1415926535897931"/>
 	  <xacro:property name="wheel_width" value="0.175" />
+    <xacro:property name="wheel_radius" value="0.127" />
 	<!-- BASE FOOTPRINT -->
 	  <xacro:if value="${publish_bf}">
