Commit message: Changed planar_move gazebo plugin configuration. Robot now moves on plane in Gazebo

File: summit_xl_description/robots/summit_xls.urdf.xacro (robot description, xacro)
@@ -45,4 +45,5 @@
 	<xacro:arg name="ros_planar_move_plugin" default="true"/>
 	<xacro:arg name="gpu" default="false"/>
+	<xacro:arg name="robot_ns" default=""/>
     <xacro:macro name="summit_xl" params="prefix publish_bf hq">
 		<!-- *************** -->
@@ -89,5 +90,5 @@
    </xacro:macro>
    <xacro:if value="$(arg ros_planar_move_plugin)">
-	   <xacro:omni_steering prefix="$(arg prefix)" publish_tf="true"/>
+	   <xacro:omni_steering namespace="$(arg robot_ns)" publish_tf="true"/>
    </xacro:if>
    <xacro:summit_xl prefix="$(arg prefix)" publish_bf="true" hq="true"/>

File: summit_xl_description/urdf/bases/summit_xl_base.gazebo.xacro (robot description, xacro)
@@ -34,7 +34,7 @@
     </gazebo>
   </xacro:macro>
-  <xacro:macro name="omni_steering" params="prefix publish_tf">
+  <xacro:macro name="omni_steering" params="namespace publish_tf">
 		<gazebo>
-	    <plugin name="omni_steering" filename="libgazebo_ros_planar_move.so">
+	    <!-- <plugin name="omni_steering" filename="libgazebo_ros_planar_move.so">
 	      <commandTopic>robotnik_base_control/cmd_vel</commandTopic>
 	      <odometryTopic>robotnik_base_control/odom</odometryTopic>
@@ -43,6 +43,19 @@
 	      <robotBaseFrame>${prefix}base_footprint</robotBaseFrame>
 	      <publishTF>${publish_tf}</publishTF>
-		  <enableYAxis>false</enableYAxis>
-	    </plugin>
+		  <enableYAxis>true</enableYAxis>
+	    </plugin> -->
+		<plugin name='planar_move' filename='libgazebo_ros_planar_move.so'>
+        <ros>
+          <namespace>${namespace}</namespace>
+          <!-- <remapping>cmd_vel:=robotnik_base_control/cmd_vel</remapping>
+          <remapping>odom:=robotnik_base_control/odom</remapping> -->
+        </ros>
+        <update_rate>100</update_rate>
+        <publish_rate>100</publish_rate>
+        <publish_odom>true</publish_odom>
+        <publish_odom_tf>true</publish_odom_tf>
+        <odometry_frame>${namespace}/odom</odometry_frame>
+        <robot_base_frame>${namespace}/base_footprint</robot_base_frame>
+      </plugin>
 	  </gazebo>
   </xacro:macro>

Commit message: updated lidar, added rviz

File: summit_xl_description/robots/summit_xls.urdf.xacro (robot description, xacro)
@@ -13,4 +13,6 @@
 	<!-- Import all available sensors -->
 	<xacro:include filename="$(find robotnik_sensors)/urdf/all_sensors.urdf.xacro" />
+<!-- Import our modified sensor -->
+	<xacro:include filename="$(find summit_xl_description)/urdf/sensors/hokuyo_ust20lx_no_frame_prefix.urdf.xacro" />
 	<xacro:property name="PI" value="3.1415926535897931"/>
 	<!-- Wheel parameters -->
@@ -19,10 +21,10 @@
 	<xacro:property name="wheel_offset_y" value="0.2045" />
 	<xacro:property name="wheel_offset_z" value="0.0" />
-	<xacro:property name="front_laser_offset_x" value="0.2865"/>
-	<xacro:property name="front_laser_offset_y" value="-0.20894"/>
-	<xacro:property name="front_laser_offset_z" value="0.2973"/>
-	<xacro:property name="rear_laser_offset_x" value="-0.2865"/>
-	<xacro:property name="rear_laser_offset_y" value="0.20894"/>
-	<xacro:property name="rear_laser_offset_z" value="0.2973"/>
+	<xacro:property name="front_laser_offset_x" value="0.356"/>
+	<xacro:property name="front_laser_offset_y" value="-0.251"/>
+	<xacro:property name="front_laser_offset_z" value="0.1566"/>
+	<xacro:property name="rear_laser_offset_x" value="-0.35"/>
+	<xacro:property name="rear_laser_offset_y" value="0.251"/>
+	<xacro:property name="rear_laser_offset_z" value="0.1566"/>
 	<xacro:property name="front_ptz_camera_offset_x" value="0.308"/>
 	<xacro:property name="front_ptz_camera_offset_y" value="0.141"/>
@@ -66,14 +68,14 @@
 		</xacro:omni_wheel>
         <!-- IMU -->
-		<xacro:sensor_imu prefix="$(arg prefix)imu" parent="$(arg prefix)base_link">
+		<xacro:sensor_imu_hector prefix="$(arg prefix)imu" ns="$(arg robot_ns)" parent="$(arg prefix)base_link">
 			<origin xyz="${imu_offset_x} ${imu_offset_y} ${imu_offset_z}" rpy="0 0 0"/>
-		</xacro:sensor_imu>
+		</xacro:sensor_imu_hector>
 		<!-- SENSORS -->
-		<xacro:sensor_sick_s300 prefix="$(arg prefix)front_laser" parent="$(arg prefix)base_link" prefix_topic="front_laser" gpu="$(arg gpu)">
+		<xacro:sensor_hokuyo_ust20lx_no_frame_prefix ns="$(arg robot_ns)" prefix="front_laser" parent="base_link">
 			<origin xyz="${front_laser_offset_x} ${front_laser_offset_y} ${front_laser_offset_z}" rpy="0 ${-PI} ${3/4*PI}" />
-		</xacro:sensor_sick_s300>
-		<xacro:sensor_sick_s300 prefix="$(arg prefix)rear_laser" parent="$(arg prefix)base_link" prefix_topic="rear_laser" gpu="$(arg gpu)">
+		</xacro:sensor_hokuyo_ust20lx_no_frame_prefix>
+        <xacro:sensor_hokuyo_ust20lx_no_frame_prefix ns="$(arg robot_ns)" prefix="rear_laser" parent="base_link">
 			<origin xyz="${rear_laser_offset_x} ${rear_laser_offset_y} ${rear_laser_offset_z}" rpy="0 ${-PI} ${-1/4*PI}" />
-		</xacro:sensor_sick_s300>
+		</xacro:sensor_hokuyo_ust20lx_no_frame_prefix>
 		<!--xacro:sensor_axis_m5013 prefix="$(arg prefix)front_ptz_camera" parent="$(arg prefix)base_link">
 			<origin xyz="${front_ptz_camera_offset_x} ${front_ptz_camera_offset_y} ${front_ptz_camera_offset_z}" rpy="${-PI/2} 0 0"/>
@@ -82,5 +84,5 @@
 			<origin xyz="${rear_ptz_camera_offset_x} ${rear_ptz_camera_offset_y} ${rear_ptz_camera_offset_z}" rpy="${-PI/2} 0 ${PI}"/>
 		</xacro:sensor_axis_m5013-->
-		<xacro:sensor_orbbec_astra prefix="$(arg prefix)front_rgbd_camera" parent="$(arg prefix)base_link" ns="front_rgbd_camera">
+		<xacro:sensor_orbbec_astra prefix="$(arg prefix)front_rgbd_camera" parent="$(arg prefix)base_link" ns="$(arg robot_ns)">
 			<origin xyz="${front_rgbd_camera_offset_x} ${front_rgbd_camera_offset_y} ${front_rgbd_camera_offset_z}" rpy="0 0 0"/>
 		</xacro:sensor_orbbec_astra>
